Commit message: ros: 포드를 든 채 회전 시험, 가감속 제한으로 미끄러짐 해결
계획서 9장은 물리 마찰에 맡기면 주행 중 미끄러진다며 detachable_joint 를
권한다. 재 보니 회전은 문제가 없고 급정지만 문제였다.

로봇과 포드의 상대 어긋남
  제자리 90도  @0.35 rad/s   0.0001 m / 요차 0.0010 rad
  제자리 180도 @0.9  rad/s   0.0001 m / 요차 0.0011 rad
  호 주행 0.25 m/s + 0.6     0.0001 m / 요차 0.0011 rad
  제자리 360도 @0.35 rad/s   좌표 소수점 4자리까지 동일
  0.5 m/s 에서 급정지         0.039 m   <- 여기만 밀린다

그래서 detachable_joint 대신 가감속을 제한했다. accel_lim 기본 0.4 m/s^2.
max_linear_acceleration 만 걸면 안 되고 min 쪽(감속)도 같이 걸어야 한다.
안 그러면 DiffDrive 가 속도를 즉시 0 으로 떨군다.

  가감속 한계 1.0   급정지 1회 +0.019 m,  4회 누적 +0.236 m  (쌓인다)
  가감속 한계 0.4   급정지 1회 -0.0005 m, 4회 누적 +0.0005 m (안 쌓인다)

제한 없이 급정지를 반복하면 포드가 결국 떨어진다. 0.3 m/s 에서 멈추는 데
0.75초 / 0.11 m 를 쓰는데 격자 간격이 2.5 m 라 여유가 충분하다.

detachable_joint 는 포드 18개 x 로봇 2대면 관절 36개를 미리 선언해야 한다.
이 결과면 그 복잡도를 감수할 이유가 없다. 경사나 충돌에서 문제가 나오면
그때 다시 본다.

docs/pod_spin.png 에 360도 회전 비교 사진을 넣었다.

File: ros/description/pod_bot.urdf.xacro (robot description, xacro)
@@ -45,4 +45,7 @@
   <xacro:property name="plate_z"   value="0.305"/>  <!-- 내렸을 때 플레이트 중심 -->
   <xacro:property name="lift_travel" value="0.16"/>
+  <!-- 가감속 한계 (m/s^2). 포드를 든 채 급정지하면 포드가 밀린다.
+       min 쪽(감속)을 안 걸면 DiffDrive 가 속도를 즉시 0 으로 떨군다. -->
+  <xacro:property name="accel_lim" value="1.0"/>
   <xacro:property name="deck_z"  value="0.27"/>    <!-- 차체 윗판 -->
   <xacro:property name="cam_z"   value="0.295"/>
@@ -326,5 +329,6 @@
       <wheel_separation>${2 * wheel_y}</wheel_separation>
       <wheel_radius>${wheel_r}</wheel_radius>
-      <max_linear_acceleration>1.0</max_linear_acceleration>
+      <max_linear_acceleration>${accel_lim}</max_linear_acceleration>
+      <min_linear_acceleration>${-accel_lim}</min_linear_acceleration>
       <topic>/${ns}/cmd_vel</topic>
       <odom_topic>/${ns}/odom</odom_topic>
